Commit message: Align TCP with the edge of gripper
Signed-off-by: Baoan Du <baoan.du.xj@renesas.com>

File: urdf/agilex_piper_gripper_macro.xacro (robot description, xacro)
@@ -7,5 +7,5 @@
     <xacro:property name="gripper_effort" value="10" />
     <xacro:property name="gripper_velocity" value="1" />
-    <xacro:property name="tcp_offset" value="0.1000" />
+    <xacro:property name="tcp_offset" value="0.1358" />
     <!-- Joint to attach the gripper to parent link -->
     <joint name="${prefix}gripper_base_joint" type="fixed">
