Commit message: Refactor folder structure to follow ros conventions
Signed-off-by: Baoan Du <baoan.du.xj@renesas.com>

File: urdf/agilex_piper_arm_macro.xacro (robot description, xacro)
@@ -36,14 +36,14 @@
         <origin xyz="0 0 0" rpy="0 0 0" />
         <geometry>
-          <mesh filename="package://agilex_piper_arm_description/urdf/meshes/base_link.STL" />
-        </geometry>
-        <material name="">
-          <color rgba="0.792156862745098 0.819607843137255 0.933333333333333 1" />
-        </material>
-      </visual>
-      <collision>
-        <origin xyz="0 0 0" rpy="0 0 0" />
-        <geometry>
-          <mesh filename="package://agilex_piper_arm_description/urdf/meshes/base_link.STL" />
+          <mesh filename="package://agilex_piper_arm_description/meshes/base_link.STL" />
+        </geometry>
+        <material name="">
+          <color rgba="0.792156862745098 0.819607843137255 0.933333333333333 1" />
+        </material>
+      </visual>
+      <collision>
+        <origin xyz="0 0 0" rpy="0 0 0" />
+        <geometry>
+          <mesh filename="package://agilex_piper_arm_description/meshes/base_link.STL" />
         </geometry>
       </collision>
@@ -60,14 +60,14 @@
         <origin xyz="0 0 0" rpy="0 0 0" />
         <geometry>
-          <mesh filename="package://agilex_piper_arm_description/urdf/meshes/link1.STL" />
-        </geometry>
-        <material name="">
-          <color rgba="0.792156862745098 0.819607843137255 0.933333333333333 1" />
-        </material>
-      </visual>
-      <collision>
-        <origin xyz="0 0 0" rpy="0 0 0" />
-        <geometry>
-          <mesh filename="package://agilex_piper_arm_description/urdf/meshes/link1.STL" />
+          <mesh filename="package://agilex_piper_arm_description/meshes/link1.STL" />
+        </geometry>
+        <material name="">
+          <color rgba="0.792156862745098 0.819607843137255 0.933333333333333 1" />
+        </material>
+      </visual>
+      <collision>
+        <origin xyz="0 0 0" rpy="0 0 0" />
+        <geometry>
+          <mesh filename="package://agilex_piper_arm_description/meshes/link1.STL" />
         </geometry>
       </collision>
@@ -93,14 +93,14 @@
         <origin xyz="0 0 0" rpy="0 0 0" />
         <geometry>
-          <mesh filename="package://agilex_piper_arm_description/urdf/meshes/link2.STL" />
-        </geometry>
-        <material name="">
-          <color rgba="0.792156862745098 0.819607843137255 0.933333333333333 1" />
-        </material>
-      </visual>
-      <collision>
-        <origin xyz="0 0 0" rpy="0 0 0" />
-        <geometry>
-          <mesh filename="package://agilex_piper_arm_description/urdf/meshes/link2.STL" />
+          <mesh filename="package://agilex_piper_arm_description/meshes/link2.STL" />
+        </geometry>
+        <material name="">
+          <color rgba="0.792156862745098 0.819607843137255 0.933333333333333 1" />
+        </material>
+      </visual>
+      <collision>
+        <origin xyz="0 0 0" rpy="0 0 0" />
+        <geometry>
+          <mesh filename="package://agilex_piper_arm_description/meshes/link2.STL" />
         </geometry>
       </collision>
@@ -126,14 +126,14 @@
         <origin xyz="0 0 0" rpy="0 0 0" />
         <geometry>
-          <mesh filename="package://agilex_piper_arm_description/urdf/meshes/link3.STL" />
-        </geometry>
-        <material name="">
-          <color rgba="0.792156862745098 0.819607843137255 0.933333333333333 1" />
-        </material>
-      </visual>
-      <collision>
-        <origin xyz="0 0 0" rpy="0 0 0" />
-        <geometry>
-          <mesh filename="package://agilex_piper_arm_description/urdf/meshes/link3.STL" />
+          <mesh filename="package://agilex_piper_arm_description/meshes/link3.STL" />
+        </geometry>
+        <material name="">
+          <color rgba="0.792156862745098 0.819607843137255 0.933333333333333 1" />
+        </material>
+      </visual>
+      <collision>
+        <origin xyz="0 0 0" rpy="0 0 0" />
+        <geometry>
+          <mesh filename="package://agilex_piper_arm_description/meshes/link3.STL" />
         </geometry>
       </collision>
@@ -159,14 +159,14 @@
         <origin xyz="0 0 0" rpy="0 0 0" />
         <geometry>
-          <mesh filename="package://agilex_piper_arm_description/urdf/meshes/link4.STL" />
-        </geometry>
-        <material name="">
-          <color rgba="0.792156862745098 0.819607843137255 0.933333333333333 1" />
-        </material>
-      </visual>
-      <collision>
-        <origin xyz="0 0 0" rpy="0 0 0" />
-        <geometry>
-          <mesh filename="package://agilex_piper_arm_description/urdf/meshes/link4.STL" />
+          <mesh filename="package://agilex_piper_arm_description/meshes/link4.STL" />
+        </geometry>
+        <material name="">
+          <color rgba="0.792156862745098 0.819607843137255 0.933333333333333 1" />
+        </material>
+      </visual>
+      <collision>
+        <origin xyz="0 0 0" rpy="0 0 0" />
+        <geometry>
+          <mesh filename="package://agilex_piper_arm_description/meshes/link4.STL" />
         </geometry>
       </collision>
@@ -192,14 +192,14 @@
         <origin xyz="0 0 0" rpy="0 0 0" />
         <geometry>
-          <mesh filename="package://agilex_piper_arm_description/urdf/meshes/link5.STL" />
-        </geometry>
-        <material name="">
-          <color rgba="0.792156862745098 0.819607843137255 0.933333333333333 1" />
-        </material>
-      </visual>
-      <collision>
-        <origin xyz="0 0 0" rpy="0 0 0" />
-        <geometry>
-          <mesh filename="package://agilex_piper_arm_description/urdf/meshes/link5.STL" />
+          <mesh filename="package://agilex_piper_arm_description/meshes/link5.STL" />
+        </geometry>
+        <material name="">
+          <color rgba="0.792156862745098 0.819607843137255 0.933333333333333 1" />
+        </material>
+      </visual>
+      <collision>
+        <origin xyz="0 0 0" rpy="0 0 0" />
+        <geometry>
+          <mesh filename="package://agilex_piper_arm_description/meshes/link5.STL" />
         </geometry>
       </collision>
@@ -225,5 +225,5 @@
         <origin xyz="0 0 0" rpy="0 0 0" />
         <geometry>
-          <mesh filename="package://agilex_piper_arm_description/urdf/meshes/link6.STL" />
+          <mesh filename="package://agilex_piper_arm_description/meshes/link6.STL" />
         </geometry>
         <material name="">
@@ -234,5 +234,5 @@
         <origin xyz="0 0 0" rpy="0 0 0" />
         <geometry>
-          <mesh filename="package://agilex_piper_arm_description/urdf/meshes/link6.STL" />
+          <mesh filename="package://agilex_piper_arm_description/meshes/link6.STL" />
         </geometry>
       </collision>

File: urdf/agilex_piper_gripper_macro.xacro (robot description, xacro)
@@ -25,5 +25,5 @@
         <origin xyz="0 0 0" rpy="0 0 0" />
         <geometry>
-          <mesh filename="package://agilex_piper_arm_description/urdf/meshes/gripper_base.STL" />
+          <mesh filename="package://agilex_piper_arm_description/meshes/gripper_base.STL" />
         </geometry>
         <material name="">
@@ -34,5 +34,5 @@
         <origin xyz="0 0 0" rpy="0 0 0" />
         <geometry>
-          <mesh filename="package://agilex_piper_arm_description/urdf/meshes/gripper_base.STL" />
+          <mesh filename="package://agilex_piper_arm_description/meshes/gripper_base.STL" />
         </geometry>
       </collision>
@@ -49,5 +49,5 @@
         <origin xyz="0 0 0" rpy="0 0 0" />
         <geometry>
-          <mesh filename="package://agilex_piper_arm_description/urdf/meshes/link7.STL" />
+          <mesh filename="package://agilex_piper_arm_description/meshes/link7.STL" />
         </geometry>
         <material name="">
@@ -58,5 +58,5 @@
         <origin xyz="0 0 0" rpy="0 0 0" />
         <geometry>
-          <mesh filename="package://agilex_piper_arm_description/urdf/meshes/link7.STL" />
+          <mesh filename="package://agilex_piper_arm_description/meshes/link7.STL" />
         </geometry>
       </collision>
@@ -82,5 +82,5 @@
         <origin xyz="0 0 0" rpy="0 0 0" />
         <geometry>
-          <mesh filename="package://agilex_piper_arm_description/urdf/meshes/link8.STL" />
+          <mesh filename="package://agilex_piper_arm_description/meshes/link8.STL" />
         </geometry>
         <material name="">
@@ -91,5 +91,5 @@
         <origin xyz="0 0 0" rpy="0 0 0" />
         <geometry>
-          <mesh filename="package://agilex_piper_arm_description/urdf/meshes/link8.STL" />
+          <mesh filename="package://agilex_piper_arm_description/meshes/link8.STL" />
         </geometry>
       </collision>

File: urdf/reference/agilex_piper_arm_ref.urdf (robot description, URDF)
Before this commit: robot piper, 7 links, 6 joints
Links:
- link base_link: geometry collision mesh filename=package://agilex_piper_urdf/meshes/base_link.STL; visual mesh filename=package://agilex_piper_urdf/meshes/base_link.STL
- link link1: geometry collision mesh filename=package://agilex_piper_urdf/meshes/link1.STL; visual mesh filename=package://agilex_piper_urdf/meshes/link1.STL
- link link2: geometry collision mesh filename=package://agilex_piper_urdf/meshes/link2.STL; visual mesh filename=package://agilex_piper_urdf/meshes/link2.STL
- link link3: geometry collision mesh filename=package://agilex_piper_urdf/meshes/link3.STL; visual mesh filename=package://agilex_piper_urdf/meshes/link3.STL
- link link4: geometry collision mesh filename=package://agilex_piper_urdf/meshes/link4.STL; visual mesh filename=package://agilex_piper_urdf/meshes/link4.STL
- link link5: geometry collision mesh filename=package://agilex_piper_urdf/meshes/link5.STL; visual mesh filename=package://agilex_piper_urdf/meshes/link5.STL
- link link6: geometry collision mesh filename=package://agilex_piper_urdf/meshes/link6.STL; visual mesh filename=package://agilex_piper_urdf/meshes/link6.STL

File: urdf/reference/agilex_piper_gripper_ref.urdf (robot description, URDF)
Before this commit: robot piper_gripper, 4 links, 3 joints
Links:
- link gripper_base: geometry collision mesh filename=package://agilex_piper_urdf/meshes/gripper_base.STL; visual mesh filename=package://agilex_piper_urdf/meshes/gripper_base.STL
- link link7: geometry collision mesh filename=package://agilex_piper_urdf/meshes/link7.STL; visual mesh filename=package://agilex_piper_urdf/meshes/link7.STL
- link link8: geometry collision mesh filename=package://agilex_piper_urdf/meshes/link8.STL; visual mesh filename=package://agilex_piper_urdf/meshes/link8.STL

Commit message: Update URDF parameters to latest specification
Signed-off-by: Dat Nguyen <dat.nguyen.dn@bp.renesas.com>

File: urdf/agilex_piper_arm_macro.xacro (robot description, xacro)
@@ -27,10 +27,9 @@
     <!-- Base Link -->
     <link name="${prefix}base_link">
-      <inertial>
-        <origin xyz="-0.00473641164191482 2.56829134630247E-05 0.041451518036016" rpy="0 0 0" />
-        <mass value="1.02" />
-        <inertia ixx="0.00267433" ixy="-0.00000073" ixz="-0.00017389"
-                 iyy="0.00282612" iyz="0.0000004" izz="0.00089624" />
-      </inertial>
+    <inertial>
+            <origin xyz="-0.00473641164191482 2.56829134630247E-05 0.041451518036016" rpy="0 0 0" />
+            <mass value="1.02" />
+            <inertia ixx="0.00267433" ixy="-0.00000073" ixz="-0.00017389" iyy="0.00282612" iyz="0.0000004" izz="0.00089624" />
+    </inertial>
       <visual>
         <origin xyz="0 0 0" rpy="0 0 0" />
@@ -52,8 +51,7 @@
     <link name="${prefix}link1">
       <inertial>
-        <origin xyz="0.00032 -0.00041 -0.00348" rpy="0 0 0" />
-        <mass value="0.71" />
-        <inertia ixx="0.00050027" ixy="0.00000078" ixz="0.00000626"
-                 iyy="0.00040879" iyz="0.00000462" izz="0.00045802" />
+              <origin xyz="0.000121504734057468 0.000104632162460536 -0.00438597309559853" rpy="0 0 0" />
+              <mass value="0.71" />
+              <inertia ixx="0.00048916" ixy="-0.00000036" ixz="-0.00000224" iyy="0.00040472" iyz="-0.00000242" izz="0.00043982" />
       </inertial>
       <visual>
@@ -85,8 +83,7 @@
     <link name="${prefix}link2">
       <inertial>
-        <origin xyz="0.21852 -0.00861 0.00126" rpy="0 0 0" />
-        <mass value="1.16" />
-        <inertia ixx="0.00111915" ixy="0.00182916" ixz="0.00019233"
-                 iyy="0.06763251" iyz="0.00000767" izz="0.067559" />
+              <origin xyz="0.198666145229743 -0.010926924140076 0.00142121714502687" rpy="0 0 0" />
+              <mass value="1.17" />
+              <inertia ixx="0.00116918" ixy="-0.00180037" ixz="0.00025146" iyy="0.06785384" iyz="-0.00000455" izz="0.06774489" />
       </inertial>
       <visual>
@@ -118,8 +115,7 @@
     <link name="${prefix}link3">
       <inertial>
-        <origin xyz="-0.01999 -0.14808 -0.00053" rpy="0 0 0" />
-        <mass value="0.5" />
-        <inertia ixx="0.01347608" ixy="0.00161034" ixz="0.00000066"
-                 iyy="0.00046377" iyz="0.00000162" izz="0.01363321" />
+              <origin xyz="-0.0202737662122021 -0.133914995944595 -0.000458682652737356" rpy="0 0 0" />
+              <mass value="0.5" />
+              <inertia ixx="0.01361711" ixy="0.00165794" ixz="-0.00000048" iyy="0.00045024" iyz="-0.00000045" izz="0.01380322" />
       </inertial>
       <visual>
@@ -150,10 +146,9 @@
     <!-- Link 4 -->
     <link name="${prefix}link4">
-      <inertial>
-        <origin xyz="0.00013 -0.00076 -0.00394" rpy="0 0 0" />
-        <mass value="0.38" />
-        <inertia ixx="0.00017844" ixy="0.00000062" ixz="0.00000067"
-                 iyy="0.00018914" iyz="0.00000408" izz="0.00014613" />
-      </inertial>
+    <inertial>
+            <origin xyz="-9.66635791618542E-05 0.000876064475651083 -0.00496880904640868" rpy="0 0 0" />
+            <mass value="0.38" />
+            <inertia ixx="0.00018501" ixy="0.00000054" ixz="0.00000120" iyy="0.00018965" iyz="-0.00000841" izz="0.00015484" />
+    </inertial>
       <visual>
         <origin xyz="0 0 0" rpy="0 0 0" />
@@ -183,10 +178,9 @@
     <!-- Link 5 -->
     <link name="${prefix}link5">
-      <inertial>
-        <origin xyz="0.00018 -0.06104 -0.00227" rpy="0 0 0" />
-        <mass value="0.39" />
-        <inertia ixx="0.00172318" ixy="0.00000259" ixz="0.00000010"
-                 iyy="0.00017936" iyz="0.00000990" izz="0.00171172" />
-      </inertial>
+    <inertial>
+            <origin xyz="-4.10554118924211E-05 -0.0566486692356075 -0.0037205791677906" rpy="0 0 0" />
+            <mass value="0.383" />
+            <inertia ixx="0.00166169" ixy="0.00000006" ixz="-0.00000007" iyy="0.00018510" iyz="0.00001026" izz="0.00164321" />
+    </inertial>
       <visual>
         <origin xyz="0 0 0" rpy="0 0 0" />
@@ -216,10 +210,9 @@
     <!-- Link 6 (End Effector) -->
     <link name="${prefix}link6">
-      <inertial>
-        <origin xyz="-0.00003 0.00006 0.04618" rpy="0 0 0" />
-        <mass value="0.46" />
-        <inertia ixx="0.00152112" ixy="0.00000202" ixz="0.00000261"
-                 iyy="0.00138626" iyz="0.00000002" izz="0.00031152" />
-      </inertial>
+    <inertial>
+            <origin xyz="-8.82590762930069E-05 9.0598378529832E-06 -0.002" rpy="0 0 0" />
+            <mass value="0.00699089613564366" />
+            <inertia ixx="5.73015540542155E-07" ixy="-1.98305403089247E-22" ixz="-7.2791893904596E-23" iyy="5.73015540542155E-07" iyz="-3.4146026640245E-24" izz="1.06738869138926E-06" />
+    </inertial>
       <visual>
         <origin xyz="0 0 0" rpy="0 0 0" />

Commit message: Revert "Update URDF parameters to latest specification"
This reverts commit cd3563b277d5b94c75be58d1c6a71ba49aaf20f0

File: urdf/agilex_piper_arm_macro.xacro (robot description, xacro)
@@ -27,9 +27,10 @@
     <!-- Base Link -->
     <link name="${prefix}base_link">
-    <inertial>
-            <origin xyz="-0.00473641164191482 2.56829134630247E-05 0.041451518036016" rpy="0 0 0" />
-            <mass value="1.02" />
-            <inertia ixx="0.00267433" ixy="-0.00000073" ixz="-0.00017389" iyy="0.00282612" iyz="0.0000004" izz="0.00089624" />
-    </inertial>
+      <inertial>
+        <origin xyz="-0.00473641164191482 2.56829134630247E-05 0.041451518036016" rpy="0 0 0" />
+        <mass value="1.02" />
+        <inertia ixx="0.00267433" ixy="-0.00000073" ixz="-0.00017389"
+                 iyy="0.00282612" iyz="0.0000004" izz="0.00089624" />
+      </inertial>
       <visual>
         <origin xyz="0 0 0" rpy="0 0 0" />
@@ -51,7 +52,8 @@
     <link name="${prefix}link1">
       <inertial>
-              <origin xyz="0.000121504734057468 0.000104632162460536 -0.00438597309559853" rpy="0 0 0" />
-              <mass value="0.71" />
-              <inertia ixx="0.00048916" ixy="-0.00000036" ixz="-0.00000224" iyy="0.00040472" iyz="-0.00000242" izz="0.00043982" />
+        <origin xyz="0.00032 -0.00041 -0.00348" rpy="0 0 0" />
+        <mass value="0.71" />
+        <inertia ixx="0.00050027" ixy="0.00000078" ixz="0.00000626"
+                 iyy="0.00040879" iyz="0.00000462" izz="0.00045802" />
       </inertial>
       <visual>
@@ -83,7 +85,8 @@
     <link name="${prefix}link2">
       <inertial>
-              <origin xyz="0.198666145229743 -0.010926924140076 0.00142121714502687" rpy="0 0 0" />
-              <mass value="1.17" />
-              <inertia ixx="0.00116918" ixy="-0.00180037" ixz="0.00025146" iyy="0.06785384" iyz="-0.00000455" izz="0.06774489" />
+        <origin xyz="0.21852 -0.00861 0.00126" rpy="0 0 0" />
+        <mass value="1.16" />
+        <inertia ixx="0.00111915" ixy="0.00182916" ixz="0.00019233"
+                 iyy="0.06763251" iyz="0.00000767" izz="0.067559" />
       </inertial>
       <visual>
@@ -115,7 +118,8 @@
     <link name="${prefix}link3">
       <inertial>
-              <origin xyz="-0.0202737662122021 -0.133914995944595 -0.000458682652737356" rpy="0 0 0" />
-              <mass value="0.5" />
-              <inertia ixx="0.01361711" ixy="0.00165794" ixz="-0.00000048" iyy="0.00045024" iyz="-0.00000045" izz="0.01380322" />
+        <origin xyz="-0.01999 -0.14808 -0.00053" rpy="0 0 0" />
+        <mass value="0.5" />
+        <inertia ixx="0.01347608" ixy="0.00161034" ixz="0.00000066"
+                 iyy="0.00046377" iyz="0.00000162" izz="0.01363321" />
       </inertial>
       <visual>
@@ -146,9 +150,10 @@
     <!-- Link 4 -->
     <link name="${prefix}link4">
-    <inertial>
-            <origin xyz="-9.66635791618542E-05 0.000876064475651083 -0.00496880904640868" rpy="0 0 0" />
-            <mass value="0.38" />
-            <inertia ixx="0.00018501" ixy="0.00000054" ixz="0.00000120" iyy="0.00018965" iyz="-0.00000841" izz="0.00015484" />
-    </inertial>
+      <inertial>
+        <origin xyz="0.00013 -0.00076 -0.00394" rpy="0 0 0" />
+        <mass value="0.38" />
+        <inertia ixx="0.00017844" ixy="0.00000062" ixz="0.00000067"
+                 iyy="0.00018914" iyz="0.00000408" izz="0.00014613" />
+      </inertial>
       <visual>
         <origin xyz="0 0 0" rpy="0 0 0" />
@@ -178,9 +183,10 @@
     <!-- Link 5 -->
     <link name="${prefix}link5">
-    <inertial>
-            <origin xyz="-4.10554118924211E-05 -0.0566486692356075 -0.0037205791677906" rpy="0 0 0" />
-            <mass value="0.383" />
-            <inertia ixx="0.00166169" ixy="0.00000006" ixz="-0.00000007" iyy="0.00018510" iyz="0.00001026" izz="0.00164321" />
-    </inertial>
+      <inertial>
+        <origin xyz="0.00018 -0.06104 -0.00227" rpy="0 0 0" />
+        <mass value="0.39" />
+        <inertia ixx="0.00172318" ixy="0.00000259" ixz="0.00000010"
+                 iyy="0.00017936" iyz="0.00000990" izz="0.00171172" />
+      </inertial>
       <visual>
         <origin xyz="0 0 0" rpy="0 0 0" />
@@ -210,9 +216,10 @@
     <!-- Link 6 (End Effector) -->
     <link name="${prefix}link6">
-    <inertial>
-            <origin xyz="-8.82590762930069E-05 9.0598378529832E-06 -0.002" rpy="0 0 0" />
-            <mass value="0.00699089613564366" />
-            <inertia ixx="5.73015540542155E-07" ixy="-1.98305403089247E-22" ixz="-7.2791893904596E-23" iyy="5.73015540542155E-07" iyz="-3.4146026640245E-24" izz="1.06738869138926E-06" />
-    </inertial>
+      <inertial>
+        <origin xyz="-0.00003 0.00006 0.04618" rpy="0 0 0" />
+        <mass value="0.46" />
+        <inertia ixx="0.00152112" ixy="0.00000202" ixz="0.00000261"
+                 iyy="0.00138626" iyz="0.00000002" izz="0.00031152" />
+      </inertial>
       <visual>
         <origin xyz="0 0 0" rpy="0 0 0" />
